File: 0015_Ethernet_Module_W5500.kicad_sch (KiCad schematic)
At the start: 39 parts, among them J1 RJ45_LED, U1 W5500, Y1 Crystal_GND24

Commit message: Add files via upload
Parts:
- added D1: LED, LED_SMD:LED_0805_2012Metric, symbol Device:LED
- added R7: 470r, Resistor_SMD:R_0805_2012Metric, symbol Device:R
- added U2: ~, Moduler_:pin_header_5-3, symbol moduler_pin:air
- J1: footprint RJ45:HANRUN_HR911105A -> Connector_RJ:RJ45_Hanrun_HR911105A
Connections:
- net +3V3: now also R7.1, U2.8
- net GND: now also D1.1 (K), U2.9
- net INT: now also U2.12
- net MISO: now also U2.2
- net MOSI: now also U2.1
- net SCS: now also U2.3
- net SLCK: now also U2.4
- net at C17.2, R11.1, R14.1: no longer C16.2, R10.1, R12.1
- new net: C16.2, R10.1, R12.1
- new net: D1.2 (A), R7.2
- no-connect marks 10 -> 21
Other:
- note added: "AIR PIN"
- note added: "SENSOR"
- moved on the sheet: C1, C10, C11, C12, C13, C14, C15, C16, C17, C2, C3, C4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
